File: kicad/solar-tracker/solar-tracker.kicad_pcb (KiCad board)
At the start: 2 copper layers, 17 parts, among them J1 Barrel_Jack_Switch, J2 Conn_01x08_Pin, J3 Conn_01x08_Pin, M1 Motor_Servo, M2 Motor_Servo

Commit message: update
Parts:
- removed DS1: ~, arduino_modulos:DS1307_RTC_MODULE
- removed LM1: ~, arduino_modulos:LM2596_Step_Down_module
- removed TCS1: ~, Connector_PinHeader_2.54mm:PinHeader_1x07_P2.54mm_Vertical
- added DS1307: ~, arduino_modulos:DS1307_RTC_MODULE, F.Cu at (36.0, 108.1)
- added LM2596: ~, arduino_modulos:LM2596_Step_Down_module, F.Cu at (28.6, 79.1)
- added TCS34725: ~, solar_tracker:TSC34725_RGB_SENSOR, F.Cu at (156.5, 74.6)
- A1: footprint Module:Arduino_Nano -> solar_tracker:Arduino_Nano
- M1, M2: footprint Connector_PinHeader_2.54mm:PinHeader_1x03_P2.54mm_Vertical -> solar_tracker:PinHeader_1x03_P2.54mm_Vertical
- R1: value LDR03 -> LDR01; footprint OptoDevice:R_LDR_10x8.5mm_P7.6mm_Vertical -> solar_tracker:R_LDR_5.1x4.3mm_P3.4mm_Vertical
- R2: value LDR03 -> LDR02; footprint OptoDevice:R_LDR_10x8.5mm_P7.6mm_Vertical -> solar_tracker:R_LDR_5.1x4.3mm_P3.4mm_Vertical
- R3: footprint OptoDevice:R_LDR_10x8.5mm_P7.6mm_Vertical -> solar_tracker:R_LDR_5.1x4.3mm_P3.4mm_Vertical
- R4: value LDR03 -> LDR04; footprint OptoDevice:R_LDR_10x8.5mm_P7.6mm_Vertical -> solar_tracker:R_LDR_5.1x4.3mm_P3.4mm_Vertical
- moved R4 76.5 mm to (179.0, 62.6), turned to -90 degrees
- moved M2 69.8 mm to (55.2, 46.8), turned to 180 degrees
- moved R3 66.7 mm to (168.2, 52.2), turned to 180 degrees
- moved M1 64.3 mm to (59.5, 46.8), turned to 180 degrees
- moved R2 59.4 mm to (166.4, 80.1), turned to 90 degrees
- moved R8 57.2 mm to (57.1, 61.2)
- moved R7 56.8 mm to (57.1, 58.1)
- moved R6 56.3 mm to (57.2, 55.0)
- moved R5 55.7 mm to (57.3, 51.9)
- moved J1 46.8 mm to (77.4, 46.1), turned to -90 degrees
- moved R1 45.9 mm to (153.7, 62.3), turned to -90 degrees
- moved J2 39.2 mm to (157.7, 47.0), turned to 90 degrees
- moved A1 35.7 mm to (70.8, 66.2)
- moved J3 28.7 mm to (68.4, 59.5), turned to 90 degrees
Connections:
- A1 pad 12: Net-(A1-D9) -> unconnected-(A1-D9-Pad12)
- A1 pad 13: Net-(A1-D10) -> unconnected-(A1-D10-Pad13)
- A1 pad 29: unconnected-(A1-GND-Pad29) -> GND
- A1 pad 8: unconnected-(A1-D5-Pad8) -> Net-(A1-D5)
- A1 pad 9: unconnected-(A1-D6-Pad9) -> Net-(A1-D6)
- J1 pad 2: Net-(LM1-IN-) -> GND
- J1 pad 3: Net-(LM1-IN-) -> GND
- J2 pad 1: +3V3 -> GND
- J2 pad 2: GND -> +3V3
- J2 pad 3: /Placa_sensor/SCL -> /Placa_sensor/LDR1
- J2 pad 4: /Placa_sensor/SDA -> /Placa_sensor/LDR2
- J2 pad 5: /Placa_sensor/LDR1 -> /Placa_sensor/LDR3
- J2 pad 6: /Placa_sensor/LDR2 -> /Placa_sensor/LDR4
- J2 pad 7: /Placa_sensor/LDR3 -> /Placa_sensor/SDA
- J2 pad 8: /Placa_sensor/LDR4 -> /Placa_sensor/SCL
- J3 pad 1: +3V3 -> GND
- J3 pad 2: GND -> +3V3
- J3 pad 3: /Placa_sensor/SCL -> /Placa_sensor/LDR1
- J3 pad 4: /Placa_sensor/SDA -> /Placa_sensor/LDR2
- J3 pad 5: /Placa_sensor/LDR1 -> /Placa_sensor/LDR3
- J3 pad 6: /Placa_sensor/LDR2 -> /Placa_sensor/LDR4
- J3 pad 7: /Placa_sensor/LDR3 -> /Placa_sensor/SDA
- J3 pad 8: /Placa_sensor/LDR4 -> /Placa_sensor/SCL
- M1 pad 1: Net-(A1-D9) -> Net-(A1-D5)
- M2 pad 1: Net-(A1-D10) -> Net-(A1-D6)
Routing:
- net GND: track 0.00 -> 294.2 mm
- net /Placa_sensor/LDR2: track 0.00 -> 121.3 mm
- net /Placa_sensor/SCL: track 0.00 -> 120.1 mm
- net /Placa_sensor/SDA: track 0.00 -> 117.6 mm
- net +3V3: track 0.00 -> 110.2 mm, vias 0 -> 2
- net +5V: track 0.00 -> 98.3 mm
- net /Placa_sensor/LDR1: track 0.00 -> 88.9 mm
- net /Placa_sensor/LDR4: track 0.00 -> 86.2 mm
- net /Placa_sensor/LDR3: track 0.00 -> 61.5 mm
- net Net-(A1-D6): track 0.00 -> 47.7 mm
- net Net-(A1-D5): track 0.00 -> 44.4 mm
- net Net-(LM2596-IN-): track 0.00 -> 43.7 mm
- added copper zone on B.Cu, net GND
Other:
- board outline added: 160.5 x 72.5 mm

Commit message: update
Parts:
- moved DS1307 2.85 mm to (38.9, 108.2)
- moved R6 1.72 mm to (58.1, 53.5)
- moved R7 1.72 mm to (58.0, 56.6)
- moved R8 1.72 mm to (58.0, 59.7)
- moved R5 1.72 mm to (58.1, 50.5)
- moved LM2596 1.28 mm to (29.6, 80.0)
- moved M1 0.73 mm to (59.5, 46.1)
- moved M2 0.73 mm to (55.2, 46.1)
Routing:
- net GND: track 294.2 -> 284.8 mm
- net /Placa_sensor/SCL: track 120.1 -> 123.0 mm
- net +3V3: track 110.2 -> 108.0 mm
- net /Placa_sensor/SDA: track 117.6 -> 115.5 mm
- net /Placa_sensor/LDR2: track 121.3 -> 119.8 mm
- net /Placa_sensor/LDR1: track 88.9 -> 87.4 mm
- net /Placa_sensor/LDR3: track 61.5 -> 60.4 mm
- net +5V: track 98.3 -> 99.3 mm
- net Net-(LM2596-IN-): track 43.7 -> 42.9 mm
- net Net-(A1-D6): track 47.7 -> 48.4 mm
Other:
- board size 160.5 x 72.5 mm -> 159.4 x 72 mm

Commit message: PCB_sensor
Parts:
- moved J2 5.05 mm to (157.0, 52.0)
- moved R3 4.45 mm to (167.7, 47.8)
- moved R1 4.16 mm to (149.5, 62.5)
- moved R4 3.48 mm to (182.5, 62.5)
- moved R2 2.42 mm to (166.0, 82.5)
- moved TCS34725 0.64 mm to (156.1, 74.2)
Connections:
- TCS34725 pad 2: GND -> unconnected-(TCS34725-INT-Pad2)
Routing:
- net GND: track 284.8 -> 441.9 mm
- net +3V3: track 108.0 -> 99.9 mm
- net /Placa_sensor/SDA: track 115.5 -> 109.9 mm
- net /Placa_sensor/LDR1: track 87.4 -> 82.2 mm
- net /Placa_sensor/LDR4: track 86.0 -> 81.7 mm
- net /Placa_sensor/LDR2: track 119.8 -> 123.3 mm
- net /Placa_sensor/SCL: track 123.0 -> 121.3 mm
- net /Placa_sensor/LDR3: track 60.4 -> 59.5 mm
Other:
- board size 159.4 x 72 mm -> 158.4 x 72 mm
