File: kicad/solar-tracker/solar-tracker.kicad_pcb (KiCad board)
At the start: 2 copper layers, 158.4 x 72 mm, 17 parts, among them J1 Barrel_Jack_Switch, J2 Conn_01x08_Pin, J3 Conn_01x08_Pin, M1 Motor_Servo, M2 Motor_Servo

Commit message: update
Parts:
- DS1307: footprint arduino_modulos:DS1307_RTC_MODULE -> solar_tracker:DS1307_RTC_MODULE
- LM2596: footprint arduino_modulos:LM2596_Step_Down_module -> solar_tracker:LM2596_Step_Down_module
- moved R4 49.6 mm to (133.2, 56.9)
- moved J2 49.6 mm to (107.7, 46.4)
- moved R1 49.6 mm to (100.2, 56.9)
- moved R2 49.6 mm to (116.7, 76.8)
- moved TCS34725 49.6 mm to (106.8, 68.5)
- moved R3 49.6 mm to (118.4, 42.1)
- moved DS1307 1.13 mm to (37.8, 108.2)
Routing:
- net GND: track 441.9 -> 440.8 mm
- net /Placa_sensor/SDA: track 109.9 -> 110.7 mm
Other:
- board size 158.4 x 72 mm -> 109.1 x 72.1 mm

Commit message: update
Parts:
- moved J2 2.85 mm to (109.8, 48.2)
- moved R4 2.18 mm to (135.4, 57.1)
- moved R1 2.18 mm to (102.4, 57.1)
- moved R2 2.18 mm to (118.9, 77.0)
- moved R3 2.18 mm to (120.6, 42.3)
- moved TCS34725 2.18 mm to (109.0, 68.7)
Routing:
- net /Placa_sensor/LDR2: track 123.3 -> 115.3 mm
- net /Placa_sensor/SCL: track 121.3 -> 115.8 mm
- net +3V3: track 99.5 -> 96.8 mm
- net /Placa_sensor/LDR3: track 59.5 -> 61.2 mm
- net /Placa_sensor/SDA: track 110.7 -> 109.0 mm
- net /Placa_sensor/LDR1: track 82.2 -> 80.5 mm
- net GND: track 440.8 -> 439.4 mm
- net /Placa_sensor/LDR4: track 81.7 -> 80.4 mm
Other:
- board size 109.1 x 72.1 mm -> 111.3 x 72 mm

Commit message: ino
Parts:
- added C1: 1uf, Capacitor_THT:CP_Radial_D6.3mm_P2.50mm, F.Cu at (134.5, 51.8)
- added C2: 1uf, Capacitor_THT:CP_Radial_D6.3mm_P2.50mm, F.Cu at (124.3, 42.4)
- added C3: 1uf, Capacitor_THT:CP_Radial_D6.3mm_P2.50mm, F.Cu at (123.9, 75.1)
- added C4: 1uf, Capacitor_THT:CP_Radial_D6.3mm_P2.50mm, F.Cu at (103.5, 52.3)
- added C5: 100UF, Capacitor_THT:CP_Radial_D6.3mm_P2.50mm, F.Cu at (85.4, 53.7)
- added C6: 100UF, Capacitor_THT:CP_Radial_D6.3mm_P2.50mm, F.Cu at (34.7, 86.9)
- added D1: 1N4007, Diode_THT:D_DO-41_SOD81_P10.16mm_Horizontal, F.Cu at (52.6, 63.8)
- DS1307: footprint solar_tracker:DS1307_RTC_MODULE -> arduino_modulos:DS1307_RTC_MODULE
- LM2596: footprint solar_tracker:LM2596_Step_Down_module -> arduino_modulos:LM2596_Step_Down_module
Connections:
- net Net-(LM2596-IN+) renamed VDD
- LM2596 pad 3: +5V -> Net-(D1-A)
Routing:
- net +3V3: track 96.8 -> 128.3 mm
- net +5V: track 99.3 -> 83.5 mm
- net /Placa_sensor/LDR2: track 115.3 -> 122.8 mm
- net Net-(D1-A): track 0.00 -> 6.75 mm
- net /Placa_sensor/LDR3: track 61.2 -> 64.9 mm
- net GND: track 439.4 -> 441.3 mm
- added copper zone on B.Cu, net VDD
