File: kicad/solar-tracker/pcb_sensor.kicad_sch (KiCad schematic)
At the start: 6 parts, among them J2 Conn_01x08_Pin

Commit message: update
Parts:
- R1: value LDR03 -> LDR01; footprint OptoDevice:R_LDR_10x8.5mm_P7.6mm_Vertical -> solar_tracker:R_LDR_5.1x4.3mm_P3.4mm_Vertical
- R2: value LDR03 -> LDR02; footprint OptoDevice:R_LDR_10x8.5mm_P7.6mm_Vertical -> solar_tracker:R_LDR_5.1x4.3mm_P3.4mm_Vertical
- R3: footprint OptoDevice:R_LDR_10x8.5mm_P7.6mm_Vertical -> solar_tracker:R_LDR_5.1x4.3mm_P3.4mm_Vertical
- R4: value LDR03 -> LDR04; footprint OptoDevice:R_LDR_10x8.5mm_P7.6mm_Vertical -> solar_tracker:R_LDR_5.1x4.3mm_P3.4mm_Vertical
- TCS34725: renamed from TCS1; footprint Connector_PinHeader_2.54mm:PinHeader_1x07_P2.54mm_Vertical -> solar_tracker:TSC34725_RGB_SENSOR
Connections:
- net 3.3V: now also J2.2 (Pin_2); no longer J2.1 (Pin_1)
- net GND: now also J2.1 (Pin_1); no longer J2.2 (Pin_2)
- net LDR1: now also J2.3 (Pin_3); no longer J2.5 (Pin_5)
- net LDR2: now also J2.4 (Pin_4); no longer J2.6 (Pin_6)
- net LDR3: now also J2.5 (Pin_5); no longer J2.7 (Pin_7)
- net LDR4: now also J2.6 (Pin_6); no longer J2.8 (Pin_8)
- net SCL: now also J2.8 (Pin_8); no longer J2.3 (Pin_3)
- net SDA: now also J2.7 (Pin_7); no longer J2.4 (Pin_4)

Commit message: PCB_sensor
Connections:
- net GND: no longer TCS34725.2 (INT)
Changed lines of the file:
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@@
-	)
-	(junction
-		(at 90.17 97.79)
-		(diameter 0)
-		(color 0 0 0 0)
 	)
 	(junction
@@
 	(wire
 		(pts
-			(xy 90.17 93.98) (xy 95.25 93.98)
-		)
-		(stroke
-			(width 0)
-			(type default)
-		)
-	)
-	(wire
-		(pts
 			(xy 96.52 60.96) (xy 96.52 57.15)
 		)
@@
 		(pts
 			(xy 39.37 85.09) (xy 50.8 85.09)
-		)
-		(stroke
-			(width 0)
-			(type default)
-		)
-	)
-	(wire
-		(pts
-			(xy 90.17 97.79) (xy 90.17 93.98)
 		)
 		(stroke
@@
 	(label "LDR4"
 		(at 44.45 87.63 0)
-		(fields_autoplaced yes)
 		(effects
 			(font
@@
 	(label "SCL"
 		(at 44.45 92.71 0)
-		(fields_autoplaced yes)
 		(effects
 			(font
@@
 	(label "LDR2"
 		(at 44.45 82.55 0)
-		(fields_autoplaced yes)
 		(effects
 			(font
@@
 	(label "LDR1"
 		(at 55.88 48.26 180)
-		(fields_autoplaced yes)
 		(effects
 			(font
@@
 	(label "LDR4"
 		(at 93.98 48.26 180)
-		(fields_autoplaced yes)
 		(effects
 			(font
@@
 	(label "LDR1"
 		(at 44.45 80.01 0)
-		(fields_autoplaced yes)
 		(effects
 			(font
@@
 	(label "SDA"
 		(at 44.45 90.17 0)
-		(fields_autoplaced yes)
 		(effects
 			(font
@@
 	(label "LDR3"
 		(at 44.45 85.09 0)
-		(fields_autoplaced yes)
 		(effects
 			(font
@@
 	(label "LDR3"
 		(at 81.28 48.26 180)
-		(fields_autoplaced yes)
 		(effects
 			(font
@@
 	(label "SCL"
 		(at 95.25 86.36 180)
-		(fields_autoplaced yes)
 		(effects
 			(font
@@
 	(label "3.3v"
 		(at 44.45 77.47 0)
-		(fields_autoplaced yes)
 		(effects
 			(font
@@
 	(label "GND"
 		(at 44.45 74.93 0)
-		(fields_autoplaced yes)
 		(effects
 			(font
@@
 	(label "LDR2"
 		(at 68.58 48.26 180)
-		(fields_autoplaced yes)
 		(effects
 			(font
@@
 	(label "SDA"
 		(at 95.25 90.17 180)
-		(fields_autoplaced yes)
 		(effects
 			(font
@@
 		(shape input)
 		(at 39.37 90.17 180)
-		(fields_autoplaced yes)
 		(effects
 			(font
@@
 		(shape input)
 		(at 39.37 80.01 180)
-		(fields_autoplaced yes)
 		(effects
 			(font
@@
 		(shape input)
 		(at 39.37 77.47 180)
-		(fields_autoplaced yes)
 		(effects
 			(font
@@
 		(shape input)
 		(at 39.37 92.71 180)
-		(fields_autoplaced yes)
 		(effects
 			(font
@@
 		(shape input)
 		(at 39.37 74.93 180)
-		(fields_autoplaced yes)
 		(effects
 			(font
@@
 		(shape input)
 		(at 39.37 85.09 180)
-		(fields_autoplaced yes)
 		(effects
 			(font
@@
 		(shape input)
 		(at 39.37 82.55 180)
-		(fields_autoplaced yes)
 		(effects
 			(font
@@
 		(shape input)
 		(at 39.37 87.63 180)
-		(fields_autoplaced yes)
-		(effects
-			(font
+		(effects
+			(font
