File: kicad/solar-tracker/solar-tracker.kicad_sch (KiCad schematic)
At the start: 2 parts, among them J1 Barrel_Jack_Switch

Commit message: update
Parts:
- added DS1: ~, arduino_modulos:DS1307_RTC_MODULE, symbol arduino_modulos:DS_1307_RTC_Module
- added J3: Conn_01x08_Pin, solar_tracker:PinHeader_1x08_P2.54mm_Vertical_large_pad, symbol solar_tracker:Conn_01x08_Pin
- added LM1: ~, arduino_modulos:LM2596_Step_Down_module, symbol arduino_modulos:LM_2596_Step_Down_Module
- added M1, M2: Motor_Servo, Connector_PinHeader_2.54mm:PinHeader_1x03_P2.54mm_Vertical, symbol Motor:Motor_Servo
- added R5, R6, R7, R8: R, solar_tracker:resistor_250mw_12mm, symbol Device:R
- J1: footprint (none) -> solar_tracker:BarrelJack_Horizontal
Connections:
- net at J1.1: now also LM1. (OUT-)
- net at J1.2: now also J1.3, LM1. (OUT-)
- net at A1.12 (D9): now also M1.1 (PWM)
- net at A1.13 (D10): now also M2.1 (PWM)
- net +3V3: now reaches A1.17 (3V3)
- net +3V3: now also DS1.3 (VCC), J3.1 (Pin_1)
- net Placa_sensor/LDR1: now reaches A1.19 (A0)
- net Placa_sensor/LDR1: now also J3.5 (Pin_5), R8.2
- net Placa_sensor/LDR2: now reaches A1.20 (A1)
- net Placa_sensor/LDR2: now also J3.6 (Pin_6), R7.2
- net Placa_sensor/LDR3: now reaches A1.21 (A2)
- net Placa_sensor/LDR3: now also J3.7 (Pin_7), R6.2
- net Placa_sensor/LDR4: now reaches A1.22 (A3)
- net Placa_sensor/LDR4: now also J3.8 (Pin_8), R5.2
- net Placa_sensor/SDA: now reaches A1.23 (A4)
- net Placa_sensor/SDA: now also DS1.4 (SDA), J3.4 (Pin_4)
- net Placa_sensor/SCL: now reaches A1.24 (A5)
- net Placa_sensor/SCL: now also DS1.5 (SCL), J3.3 (Pin_3)
- net +5V: now reaches A1.27 (+5V)
- net +5V: now also LM1. (OUT-), M1.2 (+), M2.2 (+), R5.1, R6.1, R7.1, R8.1
- net Placa_sensor/GND: now reaches A1.4 (GND)
- net Placa_sensor/GND: now also DS1.2 (GND), J3.2 (Pin_2), LM1. (OUT-), M1.3 (-), M2.3 (-)
Other:
- added sheet Placa_sensor (pcb_sensor.kicad_sch)
- moved on the sheet: A1, J1

Commit message: update
Parts:
- A1: footprint Module:Arduino_Nano -> solar_tracker:Arduino_Nano
- M1, M2: footprint Connector_PinHeader_2.54mm:PinHeader_1x03_P2.54mm_Vertical -> solar_tracker:PinHeader_1x03_P2.54mm_Vertical
- renumbered DS1 to DS1307, LM1 to LM2596
Connections:
- net +3V3: now also J3.2 (Pin_2); no longer J3.1 (Pin_1)
- net +5V: now also LM2596.3 (OUT+); no longer LM2596. (OUT-)
- net Placa_sensor/LDR1: now also J3.3 (Pin_3); no longer J3.5 (Pin_5)
- net Placa_sensor/LDR2: now also J3.4 (Pin_4); no longer J3.6 (Pin_6)
- net Placa_sensor/LDR3: now also J3.5 (Pin_5); no longer J3.7 (Pin_7)
- net Placa_sensor/LDR4: now also J3.6 (Pin_6); no longer J3.8 (Pin_8)
- net Placa_sensor/SCL: now also J3.8 (Pin_8); no longer J3.3 (Pin_3)
- net Placa_sensor/SDA: now also J3.7 (Pin_7); no longer J3.4 (Pin_4)
- net at J1.1: now also LM2596.1 (IN+); no longer LM2596. (OUT-)
- net GND: now reaches J1.2, J1.3
- net GND: now also A1.29 (GND), A1.4 (GND), DS1307.2 (GND), J3.1 (Pin_1), LM2596.2 (IN-), LM2596.4 (OUT-), M1.3 (-), M2.3 (-); no longer LM2596. (OUT-)
- net at A1.12 (D9): no longer M1.1 (PWM)
- net at A1.13 (D10): no longer M2.1 (PWM)
- net at A1.8 (D5): now also M1.1 (PWM)
- net at A1.9 (D6): now also M2.1 (PWM)
- removed net Placa_sensor/GND: A1.4 (GND), DS1307.2 (GND), J3.2 (Pin_2), LM2596. (OUT-), M1.3 (-), M2.3 (-)

Commit message: ino
Parts:
- added C1, C2, C3, C4: 1uf, Capacitor_THT:CP_Radial_D6.3mm_P2.50mm, symbol Device:C_Polarized
- added C5, C6: 100UF, Capacitor_THT:CP_Radial_D6.3mm_P2.50mm, symbol Device:C_Polarized
- added D1: 1N4007, Diode_THT:D_DO-41_SOD81_P10.16mm_Horizontal, symbol Diode:1N4007
Connections:
- net +3V3: now also C6.1
- net +5V: now also C5.1, D1.1 (K); no longer LM2596.3 (OUT+)
- net GND: now also C1.2, C2.2, C3.2, C4.2, C5.2, C6.2
- net Placa_sensor/LDR1: now also C4.1
- net Placa_sensor/LDR2: now also C3.1
- net Placa_sensor/LDR3: now also C2.1
- net Placa_sensor/LDR4: now also C1.1
- net VDD: now reaches J1.1, LM2596.1 (IN+)
- new net: D1.2 (A), LM2596.3 (OUT+)
Other:
- moved on the sheet: J1
